Commit message: Add files via upload

File: gazebo_demo/urdf/gazebo_demo.urdf.xacro (robot description, xacro)
@@ -1,4 +1,4 @@
 <?xml version="1.0" encoding="utf-8"?>
-<robot name="gazebo_demo">
+<robot name="bengine">
   <link name="base_link">
     <inertial>
@@ -88,6 +88,5 @@
     <material>Gazebo/Black</material>
   </gazebo>
-  <joint name="joint_1"
-    type="revolute">
+  <joint name="joint_1" type="revolute">
     <origin
       xyz="0 0 0.075"
@@ -117,5 +116,5 @@
   <gazebo>
     <plugin name="gazebo_ros_control" filename="libgazebo_ros_control.so">
-      <robotNamespace>/gazebo_demo</robotNamespace>
+      <robotNamespace>/bengine</robotNamespace>
       <robotSimType>gazebo_ros_control/DefaultRobotHWSim</robotSimType>
       <legacyModeNS>true</legacyModeNS>
